File: Gas_sensor_shield/Gas_sensor_shield.kicad_pcb (KiCad board)
At the start: 2 copper layers, 68.6 x 53.3 mm, 27 parts, among them J1 Gas_sensor_AIME, J2 Conn_01x08, J3 LTC1050, P1 Power, P2 Analog, P3 Digital, P4 Digital, P5 CONN_01X01, P6 CONN_01X01, P7 CONN_01X01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

Commit message: Corrections du board
Parts:
- R1, R2, R3, R4, R5, R6, R7, R8, R9: footprint Resistor_THT:R_Axial_DIN0309_L9.0mm_D3.2mm_P12.70mm_Horizontal -> Resistor_THT:R_Axial_DIN0207_L6.3mm_D2.5mm_P10.16mm_Horizontal
- moved R4 2.54 mm to (156.2, 90.5)
- moved R9 2.43 mm to (123.1, 95.2)
Connections:
- net /10 renamed /Tx(LoRa)
- net /11 renamed /Rx(LoRa)
- net /12 renamed /RST(LoRa)
- net /2 renamed /Pin_LED_ON
- net /3(**) renamed /Pin_Sensor_ON
Routing:
- net /Pin_Sensor_ON: track 61.9 -> 68.0 mm
- net Net-(C1-Pad2): track 13.6 -> 18.7 mm
- net Net-(C3-Pad2): track 11.1 -> 14.7 mm
- net /A4(SDA): track 73.2 -> 70.5 mm, vias 2 -> 0
- net Net-(J1-Pad3): track 39.2 -> 36.6 mm
- net /A0: track 11.1 -> 13.7 mm
- net /Vin=20V(on-off): track 52.6 -> 54.0 mm, vias 2 -> 4
- net /+5V(on-off): track 58.4 -> 59.5 mm, vias 1 -> 2
- net GND: vias 44 -> 54
- net (no net): vias 3 -> 2
Other:
- board text added: "PCB LOREO 10/12/20"
- board text removed: "PCB LOREO 07/12/20"
