File: Gas_sensor_shield/Gas_sensor_shield.sch (KiCad schematic (older format))
At the start: 27 parts, among them J1 Gas_sensor_AIME, J2 Conn_01x08, J3 LTC1050, P1 Power, P2 Analog, P3 Digital, P4 Digital, P5 CONN_01X01, P6 CONN_01X01, P7 CONN_01X01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

Commit message: Corrections du board
Parts:
- R1, R2, R3, R4, R5, R6, R7, R8, R9: footprint Resistor_THT:R_Axial_DIN0309_L9.0mm_D3.2mm_P12.70mm_Horizontal -> Resistor_THT:R_Axial_DIN0207_L6.3mm_D2.5mm_P10.16mm_Horizontal
Connections:
- net 10 renamed Tx(LoRa)
- net 11 renamed Rx(LoRa)
- net 12 renamed RST(LoRa)
- net 2 renamed Pin_LED_ON
- net 3(**) renamed Pin_Sensor_ON
- no-connect marks 32 -> 34
Other:
- moved on the sheet: D1, Q1, Q2, R1
